File: hardware/KiCad/output_buffer.kicad_sch (KiCad schematic)
At the start: 0 parts

Commit message: KiCad schematics on +3V3 single-supply.
Parts:
- added C10, C11, C12, C7, C8, C9: C, symbol Device:C
- added R10, R11, R12, R13, R14, R15, R16, R17: R_US, symbol Device:R_US
- added U3: MCP6022, symbol Amplifier_Operational:MCP6022
Connections:
- new net: R12.2, R13.1, U3.2 (-)
- new net: R11.2, R13.2, R14.1, U3.1
- new net: C8.2, R10.2, U3.3 (+)
- new net: C7.2, C8.1, R11.1
- new net: C9.2, U3.8 (V+)
- new net: C10.1, R14.2, R15.1
- new net: C11.1, R15.2, U3.5 (+)
- new net: C12.1, R16.2
- new net: C10.2, R16.1, U3.6 (-), U3.7
- new net +3V3: C9.1
- new net GND: C11.2, R17.2, U3.4 (V-)
- new net JACK_OUT: C12.2, R17.1
- new net SEED_OUT: C7.1
- new net VGND: R10.1, R12.1

Commit message: Input buffer simplification; removal of BAS70-04 diodes.
Parts:
- C10: value C -> 1n
- C11: value C -> 470p
- C12, C7, C8: value C -> 1µ
- C9: value C -> 0µ1
- R10: value R_US -> 5k6
- R11: value R_US -> 15k
- R12: value R_US -> 3k3
- R13: value R_US -> 10k
- R14, R15: value R_US -> 12k
- R16: value R_US -> 100R
- R17: value R_US -> 100k
Changed lines of the file:
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@@
 			)
 		)
-		(property "Value" "R_US"
+		(property "Value" "10k"
 			(at 118.11 77.47 90)
 			(show_name no)
@@
 			)
 		)
-		(property "Value" "R_US"
+		(property "Value" "5k6"
 			(at 102.87 96.5199 0)
 			(show_name no)
@@
 			)
 		)
-		(property "Value" "R_US"
+		(property "Value" "3k3"
 			(at 101.092 73.66 0)
 			(show_name no)
@@
 			)
 		)
-		(property "Value" "C"
+		(property "Value" "1µ"
 			(at 78.74 86.36 90)
 			(show_name no)
@@
 			)
 		)
-		(property "Value" "R_US"
+		(property "Value" "100k"
 			(at 217.17 118.1099 0)
 			(show_name no)
@@
 			)
 		)
-		(property "Value" "C"
+		(property "Value" "0µ1"
 			(at 124.46 119.38 90)
 			(show_name no)
@@
 			)
 		)
-		(property "Value" "R_US"
+		(property "Value" "12k"
 			(at 147.32 106.68 90)
 			(show_name no)
@@
 			)
 		)
-		(property "Value" "R_US"
+		(property "Value" "15k"
 			(at 104.394 116.586 90)
 			(show_name no)
@@
 			)
 		)
-		(property "Value" "C"
+		(property "Value" "1µ"
 			(at 205.74 107.95 90)
 			(show_name no)
@@
 			)
 		)
-		(property "Value" "R_US"
+		(property "Value" "12k"
 			(at 134.62 106.68 90)
 			(show_name no)
@@
 			)
 		)
-		(property "Value" "C"
+		(property "Value" "1n"
 			(at 160.02 95.25 90)
 			(show_name no)
@@
 			)
 		)
-		(property "Value" "C"
+		(property "Value" "1µ"
 			(at 91.44 86.36 90)
 			(show_name no)
@@
 		(in_pos_files yes)
 		(dnp no)
-		(fields_autoplaced yes)
 		(property "Reference" "R16"
 			(at 193.04 106.68 90)
@@
 			)
 		)
-		(property "Value" "R_US"
+		(property "Value" "100R"
 			(at 193.04 109.22 90)
 			(show_name no)
@@
 			)
 		)
-		(property "Value" "C"
+		(property "Value" "470p"
 			(at 163.83 119.3799 0)
 			(show_name no)

Commit message: Reduction in number of op amps from 5 to 4.
Parts:
- removed C8: 1µ, symbol Device:C
- removed R12: 3k3, symbol Device:R_US
- removed R13: 10k, symbol Device:R_US
- removed unit 1 of U3
- added unit 1 of U2
- R10: value 5k6 -> 15k
- R11: value 15k -> 150k
- renumbered C11 to C10, C12 to C11, C9 to C8, C10 to C9, R14 to R12, R15 to R13, R16 to R14, R17 to R15, U3 to U2
Connections:
- net SEED_OUT: now also C7.2; no longer C7.1
- net VGND: now also U2.3 (+); no longer R10.1
- net at R11.2, R12.1: now also U2.1
- net at R10.2: now also R11.1, U2.2 (-)
- new net: C7.1, R10.1
Other:
- moved on the sheet: C10, C11, C8, C9, R12, R13, R14, R15, U2B, U2C
