File: hardware/KiCad/schematics/power_conditioner.kicad_sch (KiCad schematic)
At the start: 3 parts

Commit message: All components fit on PCB. Some footprints replaced.
Parts:
- D3: footprint Diode_THT:D_DO-41_SOD81_P10.16mm_Horizontal -> Diode_THT:D_DO-41_SOD81_P7.62mm_Horizontal
Changed lines of the file:
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@@
 			)
 		)
-		(property "Footprint" "Diode_THT:D_DO-41_SOD81_P10.16mm_Horizontal"
+		(property "Footprint" "Diode_THT:D_DO-41_SOD81_P7.62mm_Horizontal"
 			(at 137.16 89.535 0)
 			(hide yes)
